File: PCB/ArduBoard/ArduBoard.sch (KiCad schematic (older format))
At the start: 13 parts, among them J1 Conn_01x03_Male, J2 Conn_01x12_Male, J3 Conn_01x02_Male, J4 Conn_01x08_Male, J5 Conn_01x02_Male, J6 Conn_01x02_Male, J7 Conn_01x02_Male, Q1 Q_NMOS_GDS

Commit message: Añadimos las simulaciones
Parts:
- removed D1: LED, LED_THT:LED_D5.0mm, symbol Device:LED
- removed Q1: Q_NMOS_GDS, Package_TO_SOT_THT:TO-92, symbol Device:Q_NMOS_GDS
- removed R1: 330, Resistor_THT:R_Axial_DIN0204_L3.6mm_D1.6mm_P7.62mm_Horizontal, symbol Device:R
- removed R2: 1k, Resistor_THT:R_Axial_DIN0204_L3.6mm_D1.6mm_P7.62mm_Horizontal, symbol Device:R
- removed R3: 5, Resistor_THT:R_Axial_DIN0204_L3.6mm_D1.6mm_P7.62mm_Horizontal, symbol Device:R
- added D?: LED, symbol Device:LED
- added Q?: Q_NIGBT_GCE, symbol Device:Q_NIGBT_GCE
- added Q?: Q_NMOS_GDS, symbol Device:Q_NMOS_GDS
Connections:
- net labels added: 5V, CONTROL
- wire segments 25 -> 33
Other:
- note added: "Control del led\n"
- note added: "Potencia led\n"
- note removed: "Control de potencia"
Changed lines of the file:
@@
 	1350 1050 1150 1050
 Wire Wire Line
-	2250 1650 1050 1650
+	2250 1650 1550 1650
 Wire Wire Line
 	1050 1750 2250 1750
@@
 AD7
 $Comp
-L Device:Q_NMOS_GDS Q1
-U 1 1 5B767DF3
-P 6500 1550
-F 0 "Q1" H 6705 1596 50  0000 L CNN
-F 1 "Q_NMOS_GDS" H 6705 1505 50  0000 L CNN
-F 2 "Package_TO_SOT_THT:TO-92" H 6700 1650 50  0001 C CNN
-F 3 "~" H 6500 1550 50  0001 C CNN
-	1    6500 1550
-	1    0    0    -1
-$EndComp
-$Comp
 L power:GND #PWR0103
 U 1 1 5B768349
@@
 	1    0    0    -1
 $EndComp
-$Comp
-L power:GND #PWR0104
-U 1 1 5B76843D
-P 5850 2000
-F 0 "#PWR0104" H 5850 2000 30  0001 C CNN
-F 1 "GND" H 5850 1930 30  0001 C CNN
-F 2 "" H 5850 2000 50  0001 C CNN
-F 3 "" H 5850 2000 50  0001 C CNN
-	1    5850 2000
-	1    0    0    -1
-$EndComp
-$Comp
-L Device:R R1
-U 1 1 5B768CDB
-P 5500 1550
-F 0 "R1" V 5293 1550 50  0000 C CNN
-F 1 "330" V 5384 1550 50  0000 C CNN
-F 2 "Resistor_THT:R_Axial_DIN0204_L3.6mm_D1.6mm_P7.62mm_Horizontal" V 5430 1550 50  0001 C CNN
-F 3 "~" H 5500 1550 50  0001 C CNN
-	1    5500 1550
-	0    1    1    0
-$EndComp
-$Comp
-L Device:R R2
-U 1 1 5B768D78
-P 5850 1700
-F 0 "R2" H 5920 1746 50  0000 L CNN
-F 1 "1k" H 5920 1655 50  0000 L CNN
-F 2 "Resistor_THT:R_Axial_DIN0204_L3.6mm_D1.6mm_P7.62mm_Horizontal" V 5780 1700 50  0001 C CNN
-F 3 "~" H 5850 1700 50  0001 C CNN
-	1    5850 1700
-	1    0    0    -1
-$EndComp
 Wire Wire Line
 	6600 2000 6600 1750
-Wire Wire Line
-	6300 1550 6150 1550
-Wire Wire Line
-	5850 1850 5850 2000
-Wire Wire Line
-	5850 1550 5650 1550
-Connection ~ 5850 1550
-$Comp
-L Device:R R3
-U 1 1 5B769336
-P 6600 1200
-F 0 "R3" H 6670 1246 50  0000 L CNN
-F 1 "5" H 6670 1155 50  0000 L CNN
-F 2 "Resistor_THT:R_Axial_DIN0204_L3.6mm_D1.6mm_P7.62mm_Horizontal" V 6530 1200 50  0001 C CNN
-F 3 "~" H 6600 1200 50  0001 C CNN
-	1    6600 1200
-	1    0    0    -1
-$EndComp
-Wire Wire Line
-	6600 1350 7050 1350
-Connection ~ 6600 1350
-Text GLabel 7050 1350 2    50   Input ~ 0
-LED_LOAD
 Text GLabel 5350 1550 0    50   Input ~ 0
-D2
+CONTROL
 Text GLabel 6600 750  0    50   Input ~ 0
 36V
-Wire Wire Line
-	6600 1050 6600 750
 Wire Notes Line
 	4600 600  4600 2150
@@
 Wire Notes Line
 	8750 600  4600 600
-Text Notes 6950 2100 0    118  ~ 0
-Control de potencia
+Text Notes 6250 3850 0    118  ~ 0
+Control del led\n
 $Comp
 L Connector:Conn_01x02_Male J6
@@
 	5250 1000 5100 1000
 $Comp
-L Device:LED D1
-U 1 1 5B76C6C6
-P 6150 1700
-F 0 "D1" V 6188 1583 50  0000 R CNN
-F 1 "LED" V 6097 1583 50  0000 R CNN
-F 2 "LED_THT:LED_D5.0mm" H 6150 1700 50  0001 C CNN
-F 3 "~" H 6150 1700 50  0001 C CNN
-	1    6150 1700
+L Device:Q_NIGBT_GCE Q?
+U 1 1 5B7F07C7
+P 6500 1550
+F 0 "Q?" H 6691 1596 50  0000 L CNN
+F 1 "Q_NIGBT_GCE" H 6691 1505 50  0000 L CNN
+F 2 "" H 6700 1650 50  0001 C CNN
+F 3 "~" H 6500 1550 50  0001 C CNN
+	1    6500 1550
+	1    0    0    -1
+$EndComp
+Wire Wire Line
+	5350 1550 6300 1550
+Wire Wire Line
+	6600 750  6600 1150
+Wire Wire Line
+	6600 1150 6900 1150
+Connection ~ 6600 1150
+Wire Wire Line
+	6600 1150 6600 1350
+Text GLabel 6900 1150 2    50   Input ~ 0
+LED_LOAD
+Text GLabel 6150 3250 2    50   Input ~ 0
+CONTROL
+Text GLabel 5050 3000 0    50   Input ~ 0
+D2
+$Comp
+L Device:Q_NMOS_GDS Q?
+U 1 1 5B7F2AB0
+P 5700 3000
+F 0 "Q?" H 5905 3046 50  0000 L CNN
+F 1 "Q_NMOS_GDS" H 5905 2955 50  0000 L CNN
+F 2 "" H 5900 3100 50  0001 C CNN
+F 3 "~" H 5700 3000 50  0001 C CNN
+	1    5700 3000
+	1    0    0    -1
+$EndComp
+$Comp
+L Device:LED D?
+U 1 1 5B7F2BF5
+P 5250 3250
+F 0 "D?" V 5288 3133 50  0000 R CNN
+F 1 "LED" V 5197 3133 50  0000 R CNN
+F 2 "" H 5250 3250 50  0001 C CNN
+F 3 "~" H 5250 3250 50  0001 C CNN
+	1    5250 3250
 	0    -1   -1   0
 $EndComp
-Connection ~ 6150 1550
-Wire Wire Line
-	6150 1550 5850 1550
-Wire Wire Line
-	6150 1850 6150 2000
-$Comp
-L power:GND #PWR0107
-U 1 1 5B76CA7D
-P 6150 2000
-F 0 "#PWR0107" H 6150 2000 30  0001 C CNN
-F 1 "GND" H 6150 1930 30  0001 C CNN
-F 2 "" H 6150 2000 50  0001 C CNN
-F 3 "" H 6150 2000 50  0001 C CNN
-	1    6150 2000
-	1    0    0    -1
-$EndComp
+Wire Wire Line
+	5050 3000 5250 3000
+Wire Wire Line
+	5250 3000 5250 3100
+Wire Wire Line
+	5500 3000 5250 3000
+Connection ~ 5250 3000
+$Comp
+L power:GND #PWR?
+U 1 1 5B7F3189
+P 5250 3550
+F 0 "#PWR?" H 5250 3550 30  0001 C CNN
+F 1 "GND" H 5250 3480 30  0001 C CNN
+F 2 "" H 5250 3550 50  0001 C CNN
+F 3 "" H 5250 3550 50  0001 C CNN
+	1    5250 3550
+	1    0    0    -1
+$EndComp
+Wire Wire Line
+	5250 3550 5250 3400
+$Comp
+L power:GND #PWR?
+U 1 1 5B7F354E
+P 5800 3550
+F 0 "#PWR?" H 5800 3550 30  0001 C CNN
+F 1 "GND" H 5800 3480 30  0001 C CNN
+F 2 "" H 5800 3550 50  0001 C CNN
+F 3 "" H 5800 3550 50  0001 C CNN
+	1    5800 3550
+	1    0    0    -1
+$EndComp
+Wire Wire Line
+	5800 3200 5800 3250
+Wire Wire Line
+	5800 2800 5800 2450
+Wire Wire Line
+	6150 3250 5800 3250
+Connection ~ 5800 3250
+Wire Wire Line
+	5800 3250 5800 3550
+Wire Notes Line
+	4600 2250 7650 2250
+Wire Notes Line
+	7650 2250 7650 3900
+Wire Notes Line
+	7650 3900 4600 3900
+Wire Notes Line
+	4600 3900 4600 2250
+Text Notes 7500 2050 0    118  ~ 0
+Potencia led\n
+Text GLabel 1650 1500 2    50   Input ~ 0
+5V
+Wire Wire Line
+	1650 1500 1550 1500
+Wire Wire Line
+	1550 1500 1550 1650
+Connection ~ 1550 1650
+Wire Wire Line
+	1550 1650 1050 1650
+Text GLabel 5800 2450 2    50   Input ~ 0
+5V
 $EndSCHEMATC

Commit message: Añadimos el modelo 3D del módulo
Parts:
- removed J1: Conn_01x03_Male, Connector_PinHeader_2.54mm:PinHeader_1x03_P2.54mm_Vertical, symbol Connector:Conn_01x03_Male
- removed J2: Conn_01x12_Male, Connector_PinHeader_2.54mm:PinHeader_1x12_P2.54mm_Vertical, symbol Connector:Conn_01x12_Male
- removed J4: Conn_01x08_Male, Connector_PinHeader_2.54mm:PinHeader_1x08_P2.54mm_Vertical, symbol Connector:Conn_01x08_Male
- removed J5: Conn_01x02_Male, Connector_PinHeader_2.54mm:PinHeader_1x02_P2.54mm_Vertical, symbol Connector:Conn_01x02_Male
- added J1: Conn_01x04_Male, Connector_PinHeader_2.54mm:PinHeader_1x04_P2.54mm_Vertical, symbol Connector:Conn_01x04_Male
- added J2: Conn_01x13_Male, Connector_PinHeader_2.54mm:PinHeader_1x13_P2.54mm_Vertical, symbol Connector:Conn_01x13_Male
- added J4: Conn_01x09_Male, Connector_PinHeader_2.54mm:PinHeader_1x09_P2.54mm_Vertical, symbol Connector:Conn_01x09_Male
- added J5: Conn_01x03_Male, Connector_PinHeader_2.54mm:PinHeader_1x03_P2.54mm_Vertical, symbol Connector:Conn_01x03_Male
- added R1: 500k, Resistor_THT:R_Axial_DIN0309_L9.0mm_D3.2mm_P15.24mm_Horizontal, symbol Device:R
- D1: renamed from D?; footprint (none) -> LED_THT:LED_D3.0mm
- Q1: renamed from Q?; footprint (none) -> Package_TO_SOT_THT:TO-220-3_Vertical
- Q2: renamed from Q?; footprint (none) -> Package_TO_SOT_THT:TO-247-3_Vertical
Connections:
- wire segments 33 -> 26
Changed lines of the file:
@@
 Connection ~ 2100 3200
-$Comp
-L Connector:Conn_01x03_Male J1
-U 1 1 5B759A6D
-P 850 1750
-F 0 "J1" H 956 2028 50  0000 C CNN
-F 1 "Conn_01x03_Male" H 956 1937 50  0000 C CNN
-F 2 "Connector_PinHeader_2.54mm:PinHeader_1x03_P2.54mm_Vertical" H 850 1750 50  0001 C CNN
-F 3 "~" H 850 1750 50  0001 C CNN
-	1    850  1750
-	1    0    0    -1
-$EndComp
 $Comp
 L Connector:Conn_01x02_Male J3
@@
 	1    0    0    -1
 $EndComp
-Wire Wire Line
-	2250 1550 2250 950
-Wire Wire Line
-	2250 950  1150 950
 $Comp
 L power:GND #PWR0102
 U 1 1 5B759ECA
-P 1350 1150
-F 0 "#PWR0102" H 1350 1150 30  0001 C CNN
-F 1 "GND" H 1350 1080 30  0001 C CNN
-F 2 "" H 1350 1150 50  0001 C CNN
-F 3 "" H 1350 1150 50  0001 C CNN
-	1    1350 1150
-	1    0    0    -1
-$EndComp
-Wire Wire Line
-	1350 1150 1350 1050
-Wire Wire Line
-	1350 1050 1150 1050
+P 1150 950
+F 0 "#PWR0102" H 1150 950 30  0001 C CNN
+F 1 "GND" H 1150 880 30  0001 C CNN
+F 2 "" H 1150 950 50  0001 C CNN
+F 3 "" H 1150 950 50  0001 C CNN
+	1    1150 950
+	0    -1   -1   0
+$EndComp
 Wire Wire Line
 	2250 1650 1550 1650
@@
 	1250 1850 1050 1850
 NoConn ~ 2250 2350
-$Comp
-L Connector:Conn_01x02_Male J5
-U 1 1 5B75B209
-P 3550 800
-F 0 "J5" H 3523 680 50  0000 R CNN
-F 1 "Conn_01x02_Male" H 3523 771 50  0000 R CNN
-F 2 "Connector_PinHeader_2.54mm:PinHeader_1x02_P2.54mm_Vertical" H 3550 800 50  0001 C CNN
-F 3 "~" H 3550 800 50  0001 C CNN
-	1    3550 800
-	-1   0    0    1
-$EndComp
-$Comp
-L Connector:Conn_01x12_Male J2
-U 1 1 5B75B39C
-P 850 2800
-F 0 "J2" H 956 3478 50  0000 C CNN
-F 1 "Conn_01x12_Male" H 956 3387 50  0000 C CNN
-F 2 "Connector_PinHeader_2.54mm:PinHeader_1x12_P2.54mm_Vertical" H 850 2800 50  0001 C CNN
-F 3 "~" H 850 2800 50  0001 C CNN
-	1    850  2800
-	1    0    0    -1
-$EndComp
-$Comp
-L Connector:Conn_01x08_Male J4
-U 1 1 5B75EF94
-P 1500 2950
-F 0 "J4" H 1606 3428 50  0000 C CNN
-F 1 "Conn_01x08_Male" H 1606 3337 50  0000 C CNN
-F 2 "Connector_PinHeader_2.54mm:PinHeader_1x08_P2.54mm_Vertical" H 1500 2950 50  0001 C CNN
-F 3 "~" H 1500 2950 50  0001 C CNN
-	1    1500 2950
-	1    0    0    -1
-$EndComp
 Text GLabel 3600 1150 2    50   Input ~ 0
 D0
@@
 	1    0    0    -1
 $EndComp
-Text GLabel 7900 850  2    50   Input ~ 0
+Text GLabel 7900 950  2    50   Input ~ 0
 LED_LOAD
-Text GLabel 5100 900  2    50   Input ~ 0
+Text GLabel 5100 1000 2    50   Input ~ 0
 36V
 $Comp
 L power:GND #PWR0105
 U 1 1 5B76B797
-P 5250 1050
-F 0 "#PWR0105" H 5250 1050 30  0001 C CNN
-F 1 "GND" H 5250 980 30  0001 C CNN
-F 2 "" H 5250 1050 50  0001 C CNN
-F 3 "" H 5250 1050 50  0001 C CNN
-	1    5250 1050
-	1    0    0    -1
+P 5100 900
+F 0 "#PWR0105" H 5100 900 30  0001 C CNN
+F 1 "GND" H 5100 830 30  0001 C CNN
+F 2 "" H 5100 900 50  0001 C CNN
+F 3 "" H 5100 900 50  0001 C CNN
+	1    5100 900
+	0    -1   -1   0
 $EndComp
 $Comp
 L power:GND #PWR0106
 U 1 1 5B76B916
-P 8100 1000
-F 0 "#PWR0106" H 8100 1000 30  0001 C CNN
-F 1 "GND" H 8100 930 30  0001 C CNN
-F 2 "" H 8100 1000 50  0001 C CNN
-F 3 "" H 8100 1000 50  0001 C CNN
-	1    8100 1000
-	1    0    0    -1
-$EndComp
-Wire Wire Line
-	8100 1000 8100 950
-Wire Wire Line
-	8100 950  7900 950
-Wire Wire Line
-	5250 1050 5250 1000
-Wire Wire Line
-	5250 1000 5100 1000
-$Comp
-L Device:Q_NIGBT_GCE Q?
+P 7900 850
+F 0 "#PWR0106" H 7900 850 30  0001 C CNN
+F 1 "GND" H 7900 780 30  0001 C CNN
+F 2 "" H 7900 850 50  0001 C CNN
+F 3 "" H 7900 850 50  0001 C CNN
+	1    7900 850
+	0    -1   -1   0
+$EndComp
+$Comp
+L Device:Q_NIGBT_GCE Q2
 U 1 1 5B7F07C7
 P 6500 1550
-F 0 "Q?" H 6691 1596 50  0000 L CNN
+F 0 "Q2" H 6691 1596 50  0000 L CNN
 F 1 "Q_NIGBT_GCE" H 6691 1505 50  0000 L CNN
-F 2 "" H 6700 1650 50  0001 C CNN
+F 2 "Package_TO_SOT_THT:TO-247-3_Vertical" H 6700 1650 50  0001 C CNN
 F 3 "~" H 6500 1550 50  0001 C CNN
 	1    6500 1550
@@
 D2
 $Comp
-L Device:Q_NMOS_GDS Q?
+L Device:Q_NMOS_GDS Q1
 U 1 1 5B7F2AB0
 P 5700 3000
-F 0 "Q?" H 5905 3046 50  0000 L CNN
+F 0 "Q1" H 5905 3046 50  0000 L CNN
 F 1 "Q_NMOS_GDS" H 5905 2955 50  0000 L CNN
-F 2 "" H 5900 3100 50  0001 C CNN
+F 2 "Package_TO_SOT_THT:TO-220-3_Vertical" H 5900 3100 50  0001 C CNN
 F 3 "~" H 5700 3000 50  0001 C CNN
 	1    5700 3000
@@
 $EndComp
 $Comp
-L Device:LED D?
+L Device:LED D1
 U 1 1 5B7F2BF5
 P 5250 3250
-F 0 "D?" V 5288 3133 50  0000 R CNN
+F 0 "D1" V 5288 3133 50  0000 R CNN
 F 1 "LED" V 5197 3133 50  0000 R CNN
-F 2 "" H 5250 3250 50  0001 C CNN
+F 2 "LED_THT:LED_D3.0mm" H 5250 3250 50  0001 C CNN
 F 3 "~" H 5250 3250 50  0001 C CNN
 	1    5250 3250
@@
 Connection ~ 5250 3000
 $Comp
-L power:GND #PWR?
+L power:GND #PWR0104
 U 1 1 5B7F3189
 P 5250 3550
-F 0 "#PWR?" H 5250 3550 30  0001 C CNN
+F 0 "#PWR0104" H 5250 3550 30  0001 C CNN
 F 1 "GND" H 5250 3480 30  0001 C CNN
 F 2 "" H 5250 3550 50  0001 C CNN
@@
 	5250 3550 5250 3400
 $Comp
-L power:GND #PWR?
+L power:GND #PWR0107
 U 1 1 5B7F354E
 P 5800 3550
-F 0 "#PWR?" H 5800 3550 30  0001 C CNN
+F 0 "#PWR0107" H 5800 3550 30  0001 C CNN
 F 1 "GND" H 5800 3480 30  0001 C CNN
 F 2 "" H 5800 3550 50  0001 C CNN
@@
 Wire Wire Line
 	6150 3250 5800 3250
-Connection ~ 5800 3250
-Wire Wire Line
-	5800 3250 5800 3550
 Wire Notes Line
 	4600 2250 7650 2250
@@
 Text GLabel 5800 2450 2    50   Input ~ 0
 5V
+$Comp
+L Device:R R1
+U 1 1 5B7F6974
+P 5800 3400
+F 0 "R1" H 5870 3446 50  0000 L CNN
+F 1 "500k" H 5870 3355 50  0000 L CNN
+F 2 "Resistor_THT:R_Axial_DIN0309_L9.0mm_D3.2mm_P15.24mm_Horizontal" V 5730 3400 50  0001 C CNN
+F 3 "~" H 5800 3400 50  0001 C CNN
+	1    5800 3400
+	1    0    0    -1
+$EndComp
+Connection ~ 5800 3250
+Wire Wire Line
+	2250 1550 2250 1050
+Wire Wire Line
+	2250 1050 1150 1050
+$Comp
+L Connector:Conn_01x04_Male J1
+U 1 1 5B7FCB21
+P 850 1650
+F 0 "J1" H 956 1928 50  0000 C CNN
+F 1 "Conn_01x04_Male" H 956 1837 50  0000 C CNN
+F 2 "Connector_PinHeader_2.54mm:PinHeader_1x04_P2.54mm_Vertical" H 850 1650 50  0001 C CNN
+F 3 "~" H 850 1650 50  0001 C CNN
+	1    850  1650
+	1    0    0    -1
+$EndComp
+$Comp
+L power:GND #PWR0108
+U 1 1 5B7FCDE2
+P 1050 1550
+F 0 "#PWR0108" H 1050 1550 30  0001 C CNN
+F 1 "GND" H 1050 1480 30  0001 C CNN
+F 2 "" H 1050 1550 50  0001 C CNN
+F 3 "" H 1050 1550 50  0001 C CNN
+	1    1050 1550
+	0    -1   -1   0
+$EndComp
+$Comp
+L Connector:Conn_01x13_Male J2
+U 1 1 5B7FD576
+P 850 2800
+F 0 "J2" H 956 3578 50  0000 C CNN
+F 1 "Conn_01x13_Male" H 956 3487 50  0000 C CNN
+F 2 "Connector_PinHeader_2.54mm:PinHeader_1x13_P2.54mm_Vertical" H 850 2800 50  0001 C CNN
+F 3 "~" H 850 2800 50  0001 C CNN
+	1    850  2800
+	1    0    0    -1
+$EndComp
+$Comp
+L power:GND #PWR0109
+U 1 1 5B7FD85F
+P 1050 2200
+F 0 "#PWR0109" H 1050 2200 30  0001 C CNN
+F 1 "GND" H 1050 2130 30  0001 C CNN
+F 2 "" H 1050 2200 50  0001 C CNN
+F 3 "" H 1050 2200 50  0001 C CNN
+	1    1050 2200
+	0    -1   -1   0
+$EndComp
+$Comp
+L Connector:Conn_01x09_Male J4
+U 1 1 5B7FDD18
+P 1500 2950
+F 0 "J4" H 1606 3528 50  0000 C CNN
+F 1 "Conn_01x09_Male" H 1606 3437 50  0000 C CNN
+F 2 "Connector_PinHeader_2.54mm:PinHeader_1x09_P2.54mm_Vertical" H 1500 2950 50  0001 C CNN
+F 3 "~" H 1500 2950 50  0001 C CNN
+	1    1500 2950
+	1    0    0    -1
+$EndComp
+$Comp
+L power:GND #PWR0110
+U 1 1 5B7FDDF9
+P 1700 2550
+F 0 "#PWR0110" H 1700 2550 30  0001 C CNN
+F 1 "GND" H 1700 2480 30  0001 C CNN
+F 2 "" H 1700 2550 50  0001 C CNN
+F 3 "" H 1700 2550 50  0001 C CNN
+	1    1700 2550
+	0    -1   -1   0
+$EndComp
+$Comp
+L Connector:Conn_01x03_Male J5
+U 1 1 5B7FE6BC
+P 3550 800
+F 0 "J5" H 3523 730 50  0000 R CNN
+F 1 "Conn_01x03_Male" H 3523 821 50  0000 R CNN
+F 2 "Connector_PinHeader_2.54mm:PinHeader_1x03_P2.54mm_Vertical" H 3550 800 50  0001 C CNN
+F 3 "~" H 3550 800 50  0001 C CNN
+	1    3550 800
+	-1   0    0    1
+$EndComp
+$Comp
+L power:GND #PWR0111
+U 1 1 5B7FE7E7
+P 3350 900
+F 0 "#PWR0111" H 3350 900 30  0001 C CNN
+F 1 "GND" H 3350 830 30  0001 C CNN
+F 2 "" H 3350 900 50  0001 C CNN
+F 3 "" H 3350 900 50  0001 C CNN
+	1    3350 900
+	0    1    1    0
+$EndComp
 $EndSCHEMATC
